File: latchbox-lite.brd (EAGLE design)
At the start: 59.1 x 21.8 mm, 26 parts, among them IC1 PIC12F1822SO08

Commit message: version 1 proto
Parts:
- removed TR1: (no value), microbuilder:SOT23-R
- added Q1: (no value), microbuilder:SOT23-R
- added Q2: (no value), transistor:SOT23-BEC
- added R7: (no value), rcl:R0805
- D2: value 0805DIODE -> (none); device jasons_stuff:0805DIODE -> microbuilder:SOD-123
- D3: value (none) -> 0805DIODE; device microbuilder:SOD-123 -> jasons_stuff:0805DIODE
- moved ICSP 35.1 mm to (5.21, 21.6), turned to 270 degrees
- moved R6 23.7 mm to (27.9, 22.9), turned to 90 degrees
- moved R5 17.6 mm to (33.0, 14.0), turned to 0 degrees
- moved R4 16.5 mm to (41.8, 14.0), turned to 180 degrees
- moved D1 10.5 mm to (50.8, 15.4)
- moved D2 9.00 mm to (42.8, 22.9)
- moved D4 6.35 mm to (33.0, 19.1), turned to 0 degrees
- moved D5 5.08 mm to (33.0, 16.5), turned to 0 degrees
- moved D3 4.45 mm to (38.1, 22.9)
- moved C2 3.00 mm to (10.0, 18.5)
- moved C3 2.84 mm to (58.4, 22.9)
- moved R3 2.84 mm to (41.9, 17.8), turned to 90 degrees
- moved IC1 1.94 mm to (26.0, 15.0)
- moved C1 0.68 mm to (27.7, 19.1)
- moved IN 0.25 mm to (48.3, 29.5)
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- renumbered L1 to LED1, L2 to LED2, PTC1 to F1, TR2 to Q3
Connections:
- new net N: D1.C, Q1.1, Q2.C, R4.1
- new net N$2: Q2.B, R5.1
- new net Z: D1.A, D4.A, D5.A, R2.2
- net GND: now also D3.C, Q2.E; no longer D1.C
- net INPUT: now also D5.C, IC1.2; no longer D1.A, D2.C, D5.A, IC1.3, R2.2
- net N$10: now also R7.1; no longer R6.1
- net N$11: now also R7.2; no longer R6.2
- net N$15: now also D2.A; no longer D3.A
- net N$16: now also R3.2; no longer R5.2
- net N$4: now also D2.C, Q1.2, R3.1, R4.2; no longer D3.C, R3.2, R5.1, TR1.2
- net N$6: now also R6.2; no longer R4.2
- net N$9: now also D3.A; no longer D4.A
- net OUTPUT: now also R6.1; no longer R4.1
- net POWER_CTRL: now also IC1.3, R5.2; no longer D5.C, IC1.2, R3.1, TR1.1
- net VCC: now also Q1.3; no longer D2.A, TR1.3
Routing:
- net Z: track 0.00 -> 34.1 mm, vias 0 -> 2
- net N$14: track 4.00 -> 35.4 mm, vias 0 -> 1
- net INPUT: track 34.5 -> 3.50 mm, vias 2 -> 0
- net N$11: track 54.4 -> 30.2 mm, vias 2 -> 1
- net N: track 0.00 -> 22.5 mm
- net N$4: track 54.7 -> 33.4 mm
- net N$12: track 53.4 -> 71.3 mm
- net POWER_CTRL: track 18.6 -> 3.58 mm
- net N$16: track 13.8 -> 28.7 mm
- net N$7: track 33.2 -> 41.9 mm
- net VCC: track 74.6 -> 81.5 mm, vias 3 -> 1
- net N$2: track 0.00 -> 5.27 mm
- net N$10: track 2.93 -> 5.17 mm
- net N$8: track 14.3 -> 15.9 mm
- net OUTPUT: track 13.8 -> 13.0 mm, vias 0 -> 2
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Other:
- board text added: "Latchbox"
- board text added: "USB PWR"
- board text added: "oneswitch.org.uk"
- board text added: "pcb rev 1"
- board text added: "sixty four pixels"

Commit message: sas
Parts:
- R1, R6, R7: value (none) -> 1k
- R2: value (none) -> 100r
- R4: value (none) -> 10k
Changed lines of the file:
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@@
 <attribute name="NAME" x="29.0752" y="21.506" size="1.27" layer="22" font="vector" ratio="20" rot="MR180"/>
 </element>
-<element name="R2" library="rcl" package="R0805" value="" x="48.26" y="27.305" smashed="yes" rot="MR270">
+<element name="R2" library="rcl" package="R0805" value="100r" x="48.26" y="27.305" smashed="yes" rot="MR270">
 <attribute name="NAME" x="51.689" y="25.654" size="1.27" layer="26" font="vector" ratio="20" rot="MR0"/>
 <attribute name="VALUE" x="50.8" y="27.94" size="1.27" layer="28" rot="MR270"/>
@@
 <attribute name="VALUE" x="43.18" y="33.655" size="1.27" layer="27" rot="R180"/>
 </element>
-<element name="R6" library="rcl" package="R0805" value="" x="27.94" y="22.86" smashed="yes" rot="MR90">
+<element name="R6" library="rcl" package="R0805" value="1k" x="27.94" y="22.86" smashed="yes" rot="MR90">
 <attribute name="NAME" x="26.543" y="24.13" size="1.27" layer="26" font="vector" ratio="20" rot="MR0"/>
 <attribute name="VALUE" x="25.4" y="22.225" size="1.27" layer="28" rot="MR90"/>
@@
 <attribute name="VALUE" x="55.88" y="20.193" size="1.27" layer="27" ratio="10" rot="R270"/>
 </element>
-<element name="R4" library="rcl" package="R0805" value="" x="41.783" y="13.97" smashed="yes" rot="MR180">
+<element name="R4" library="rcl" package="R0805" value="10k" x="41.783" y="13.97" smashed="yes" rot="MR180">
 <attribute name="NAME" x="40.513" y="12.827" size="1.27" layer="26" font="vector" ratio="20" rot="MR180"/>
 <attribute name="VALUE" x="41.148" y="16.51" size="1.27" layer="28" rot="MR180"/>
@@
 <attribute name="VALUE" x="10.795" y="27.559" size="1.27" layer="27" ratio="10"/>
 </element>
-<element name="R7" library="rcl" package="R0805" value="" x="10.16" y="24.257" smashed="yes" rot="MR270">
+<element name="R7" library="rcl" package="R0805" value="1k" x="10.16" y="24.257" smashed="yes" rot="MR270">
 <attribute name="NAME" x="8.89" y="27.686" size="1.27" layer="26" font="vector" ratio="20" rot="MR180"/>
 <attribute name="VALUE" x="12.7" y="24.892" size="1.27" layer="28" rot="MR270"/>
 </element>
-<element name="R1" library="rcl" package="R0805" value="" x="59.69" y="29.21" smashed="yes" rot="MR270">
+<element name="R1" library="rcl" package="R0805" value="1k" x="59.69" y="29.21" smashed="yes" rot="MR270">
 <attribute name="NAME" x="55.88" y="32.004" size="1.27" layer="26" font="vector" ratio="20" rot="MR180"/>
 <attribute name="VALUE" x="62.23" y="29.845" size="1.27" layer="28" rot="MR270"/>
