File: latchbox-lite.brd (EAGLE design)
At the start: 59.1 x 21.8 mm, 28 parts, among them IC1 PIC12F1822SO08

Commit message: v2 possible
Parts:
- removed C3: (no value), rcl:E2,5-6E
- removed Q3: (no value), transistor:SOT23-BEC
- removed R7: 1k, rcl:R0805
- added D6, D7: 0805DIODE, jasons_stuff:0805DIODE
- added S1: (no value), switch-omron:B3F-31XX
- C2: value (none) -> 4u7
- D1, D3: value 0805DIODE -> (none); device jasons_stuff:0805DIODE -> microbuilder:SOD-123
- R1: value 1k -> 100r
- R2: value 100r -> 1k
- R3: value (none) -> 10k
- R4: value 10k -> 4r7
- R5: value (none) -> 1k
- moved C2 36.3 mm to (46.0, 23.6), turned to 180 degrees
- moved F1 20.3 mm to (59.3, 19.4), turned to 270 degrees
- moved Q2 20.1 mm to (19.2, 24.5)
- moved BATT 19.3 mm to (59.3, 25.4), turned to 270 degrees
- moved R5 16.2 mm to (18.5, 21.2)
- moved D2 10.4 mm to (46.4, 13.1), turned to 0 degrees
- moved R6 10.3 mm to (18.9, 27.9), turned to 0 degrees
- moved LED2 10.1 mm to (45.8, 30.5)
- moved LED1 10.1 mm to (18.9, 30.5)
- moved D3 9.92 mm to (39.8, 13.1), turned to 180 degrees
- moved R3 9.72 mm to (51.6, 16.6), turned to 180 degrees
- moved R1 6.63 mm to (53.3, 27.3)
- moved D4 5.97 mm to (33.0, 13.1), turned to 180 degrees
- moved USB 5.72 mm to (38.1, 28.1)
- moved Q1 5.26 mm to (51.6, 13.6), turned to 180 degrees
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Connections:
- removed net N: D1.C, Q1.1, Q2.C, R4.1
- removed net N$2: Q2.B, R5.1
- new net USB_POWER: D2.A, D3.A, R4.1
- net GND: now also D6.C, D7.C, S1.1; no longer C3.-, D3.C, D4.C, Q3.E
- net N$1: now also R1.1; no longer R2.1
- net N$10: now also R6.1; no longer R7.1
- net N$11: now also R6.2; no longer R7.2
- net N$12: now also D3.C, R2.2; no longer R1.2
- net N$14: now also D4.A, S1.2
- net N$15: now also D1.A; no longer D2.A
- net N$16: now also R4.2; no longer R3.2
- net N$3: now also R2.1; no longer R1.1
- net N$4: now also D1.C, R3.2; no longer C3.+, D2.C, R3.1, R4.2
- net N$6: now also Q2.B, R5.2; no longer Q3.B, R6.2
- net N$9: now also D7.A, Q2.C; no longer D3.A, Q3.C
- net OUTPUT: now also R5.1; no longer R6.1
- net POWER_CTRL: now also D4.C, Q1.1, R3.1; no longer R5.2
- net VCC: now also D2.C
- net Z: now also D6.A, R1.2; no longer D1.A, D4.A, R2.2
Routing:
- net POWER_CTRL: track 3.58 -> 32.9 mm
- net N$4: track 33.4 -> 4.46 mm, vias 2 -> 0
- net N: track 22.5 -> 0.00 mm
- net N$14: track 35.4 -> 57.9 mm
- net N$16: track 28.7 -> 16.8 mm
- net N$9: track 5.79 -> 17.0 mm
- net VCC: track 81.5 -> 91.5 mm, vias 1 -> 2
- net Z: track 34.1 -> 24.8 mm, vias 2 -> 0
- net USB_POWER: track 0.00 -> 7.43 mm
- net N$11: track 30.2 -> 37.1 mm, vias 1 -> 0
- net N$7: track 41.9 -> 35.1 mm
- net N$2: track 5.27 -> 0.00 mm
- net N$3: track 7.07 -> 2.67 mm
- net N$8: track 15.9 -> 20.1 mm
- net GND: track 0.51 -> 4.00 mm
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Other:
- outline, holes or cut-outs redrawn
- board text added: "pcb rev 2"
- board text removed: "pcb rev 1"

Commit message: V3
Connections:
- net GND: now also IN.1; no longer IN.3
Changed lines of the file:
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@@
 <contactref element="D6" pad="C"/>
 <contactref element="BATT" pad="1"/>
-<contactref element="IN" pad="3"/>
 <contactref element="D7" pad="C"/>
 <contactref element="Q2" pad="E"/>
@@
 <vertex x="66.04" y="35.56"/>
 </polygon>
+<contactref element="IN" pad="1"/>
 </signal>
 <signal name="N$5">

Commit message: V3 BOARD
Parts:
- removed D7: 0805DIODE, jasons_stuff:0805DIODE
- added Q3: (no value), transistor:SOT23-BEC
- added R7: 10k, rcl:R0805
- moved D6 6.35 mm to (27.9, 22.9), turned to 270 degrees
- moved D3 3.45 mm to (39.4, 16.5)
- moved D4 3.43 mm to (33.0, 16.5), turned to 0 degrees
- moved D5 2.54 mm to (33.0, 19.1)
- moved R4 2.42 mm to (39.4, 19.1)
Connections:
- new net N$13: Q3.B, R7.2
- new net N$2: D3.A, Q1.1, Q3.C, R3.1
- net GND: now also D5.C, Q3.E; no longer D7.C
- net INPUT: now also D4.C; no longer D5.C
- net N$12: no longer D3.C
- net N$14: now also D3.C; no longer D4.A
- net N$9: now also D6.A; no longer D7.A
- net POWER_CTRL: now also R7.1; no longer D4.C, Q1.1, R3.1
- net USB_POWER: no longer D3.A
- net Z: now also D4.A; no longer D6.A
Routing:
- net POWER_CTRL: track 32.9 -> 3.45 mm
- net VCC: track 91.5 -> 71.2 mm, vias 2 -> 3
- net N$2: track 0.00 -> 16.1 mm
- net N$16: track 16.8 -> 11.4 mm
- net N$13: track 0.00 -> 5.11 mm
- net N$7: track 35.1 -> 39.8 mm
- net N$8: track 20.1 -> 23.5 mm, vias 0 -> 2
- net N$14: track 57.9 -> 55.1 mm, vias 1 -> 2
- net N$12: track 69.8 -> 67.6 mm, vias 3 -> 2
- net USB_POWER: track 7.43 -> 9.48 mm, vias 0 -> 2
- net OUTPUT: track 11.5 -> 12.1 mm
- net N$9: track 17.0 -> 16.5 mm
- net GND: track 4.00 -> 4.01 mm, vias 5 -> 0
Other:
- board text added: "pcb rev 3"
- board text removed: "pcb rev 2"

Commit message: V2 firmware
Parts:
- R7: value 10k -> 1k

Commit message: V4
Parts:
- D3: value (none) -> 0805DIODE; device microbuilder:SOD-123 -> jasons_stuff:0805DIODE
- moved D3 0.13 mm to (39.2, 16.5)
Connections:
- net N$14: now also D3.A; no longer D3.C
- net N$2: now also D3.C; no longer D3.A
Other:
- board text added: "pcb rev 4"
- board text removed: "pcb rev 3"
Changed lines of the file:
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@@
 <text x="25.4" y="15.367" size="1.27" layer="51" font="vector" ratio="20">sixty four pixels</text>
 <text x="25.4" y="13.843" size="1.27" layer="51" font="vector" ratio="20">oneswitch.org.uk</text>
-<text x="23.241" y="13.081" size="1.27" layer="51" font="vector" ratio="20" rot="R180">pcb rev 3</text>
+<text x="23.241" y="13.081" size="1.27" layer="51" font="vector" ratio="20" rot="R180">pcb rev 4</text>
 <wire x1="58.42" y1="33.02" x2="59.309" y2="33.02" width="0.4064" layer="20"/>
 <wire x1="59.309" y1="33.02" x2="61.849" y2="30.48" width="0.4064" layer="20"/>
@@
 <attribute name="NAME" x="32.258" y="12.954" size="1.27" layer="26" font="vector" ratio="20" rot="MR180"/>
 </element>
-<element name="D3" library="microbuilder" package="SOD-123" value="" x="39.37" y="16.51" smashed="yes" rot="MR180">
-<attribute name="NAME" x="41.91" y="17.145" size="1.27" layer="26" font="vector" ratio="20" rot="MR180"/>
-<attribute name="VALUE" x="38.1" y="18.034" size="0.4064" layer="26" rot="MR180"/>
+<element name="D3" library="jasons_stuff" package="0805DIODE" value="0805DIODE" x="39.243" y="16.51" smashed="yes" rot="MR180">
+<attribute name="NAME" x="41.74" y="15.6132" size="1.27" layer="22" font="vector" ratio="20" rot="MR90"/>
 </element>
 </elements>
@@
 <contactref element="ICSP" pad="1"/>
 <contactref element="S1" pad="2"/>
-<contactref element="D3" pad="C"/>
 <wire x1="28.6512" y1="13.081" x2="26.543" y2="13.081" width="0.4064" layer="16"/>
 <via x="26.543" y="13.081" extent="1-16" drill="0.6"/>
@@
 <wire x1="25.146" y1="26.543" x2="25.146" y2="29.718" width="0.4064" layer="1"/>
 <wire x1="25.146" y1="29.718" x2="24.2824" y2="30.5816" width="0.4064" layer="1"/>
-<wire x1="37.52" y1="16.51" x2="36.195" y2="16.51" width="0.4064" layer="16"/>
-<via x="36.195" y="16.51" extent="1-16" drill="0.6"/>
+<via x="36.576" y="16.51" extent="1-16" drill="0.6"/>
 <wire x1="23.749" y1="25.146" x2="23.749" y2="14.351" width="0.4064" layer="1"/>
 <wire x1="23.749" y1="14.351" x2="25.019" y2="13.081" width="0.4064" layer="1"/>
@@
 <wire x1="7.493" y1="26.67" x2="8.636" y2="27.813" width="0.4064" layer="1"/>
 <wire x1="8.636" y1="27.813" x2="19.177" y2="27.813" width="0.4064" layer="1"/>
-<wire x1="36.195" y1="16.51" x2="29.972" y2="16.51" width="0.4064" layer="1"/>
+<wire x1="36.576" y1="16.51" x2="29.972" y2="16.51" width="0.4064" layer="1"/>
 <wire x1="29.972" y1="16.51" x2="26.543" y2="13.081" width="0.4064" layer="1"/>
 <wire x1="19.177" y1="27.813" x2="21.844" y2="25.146" width="0.4064" layer="1"/>
 <wire x1="21.844" y1="25.146" x2="23.749" y2="25.146" width="0.4064" layer="1"/>
+<contactref element="D3" pad="A"/>
+<wire x1="36.576" y1="16.51" x2="37.9812" y2="16.51" width="0.4064" layer="16"/>
+<wire x1="37.9812" y1="16.51" x2="37.9812" y2="16.515" width="0.4064" layer="16"/>
 </signal>
 <signal name="N$11">
@@
 <contactref element="R4" pad="2"/>
 <wire x1="38.608" y1="19.238" x2="38.42" y2="19.05" width="0.4064" layer="16"/>
-<via x="36.449" y="19.05" extent="1-16" drill="0.6"/>
-<wire x1="36.449" y1="19.05" x2="38.42" y2="19.05" width="0.4064" layer="16"/>
+<via x="36.576" y="19.05" extent="1-16" drill="0.6"/>
+<wire x1="36.576" y1="19.05" x2="38.42" y2="19.05" width="0.4064" layer="16"/>
 <wire x1="38.1" y1="23.241" x2="39.4" y2="24.541" width="0.4064" layer="1"/>
 <wire x1="39.4" y1="27.017" x2="39.4" y2="24.541" width="0.4064" layer="1"/>
-<wire x1="36.449" y1="19.05" x2="36.449" y2="19.939" width="0.4064" layer="1"/>
+<wire x1="36.576" y1="19.05" x2="36.449" y2="19.939" width="0.4064" layer="1"/>
 <wire x1="36.449" y1="19.939" x2="38.1" y2="21.59" width="0.4064" layer="1"/>
 <wire x1="38.1" y1="21.59" x2="38.1" y2="23.241" width="0.4064" layer="1"/>
@@
 <contactref element="R3" pad="1"/>
 <contactref element="Q3" pad="C"/>
-<contactref element="D3" pad="A"/>
-<wire x1="41.22" y1="16.51" x2="41.22" y2="14.732" width="0.4064" layer="16"/>
 <wire x1="41.22" y1="14.732" x2="41.22" y2="14.212" width="0.4064" layer="16"/>
 <wire x1="41.22" y1="14.212" x2="40.597" y2="13.589" width="0.4064" layer="16"/>
@@
 <wire x1="49.149" y1="15.367" x2="48.514" y2="14.732" width="0.4064" layer="16"/>
 <wire x1="48.514" y1="14.732" x2="41.22" y2="14.732" width="0.4064" layer="16"/>
+<contactref element="D3" pad="C"/>
+<wire x1="41.22" y1="14.732" x2="41.22" y2="15.7762" width="0.4064" layer="16"/>
+<wire x1="41.22" y1="15.7762" x2="40.4812" y2="16.515" width="0.4064" layer="16"/>
 </signal>
 <signal name="N$13">
@@
 </signal>
 </signals>
+<errors>
+</errors>
 </board>
 </drawing>
