File: latchbox-lite.sch (EAGLE design)
At the start: 26 parts, among them IC1 PIC12F1822SO08

Commit message: version 1 proto
Parts:
- removed L1, L2: (no value), led:LED3MM
- removed TR2: (no value), transistor:MMBTA13LT1-NPN_DARL-SOT23-BEC
- added LED1, LED2: (no value), led:LED3MM
- added Q2: (no value), transistor:MMBT3904LT1-NPN-SOT23-BEC
- added Q3: (no value), transistor:MMBTA13LT1-NPN_DARL-SOT23-BEC
- added R7: (no value), rcl:R-EU_R0805
- D2: value 0805DIODE -> (none); device jasons_stuff:0805DIODE -> microbuilder:DIODESOD-123
- D3: value (none) -> 0805DIODE; device microbuilder:DIODESOD-123 -> jasons_stuff:0805DIODE
- renumbered PTC1 to F1, TR1 to Q1
Connections:
- new net N: D1.P$1, Q1.G, Q2.C, R4.1
- new net N$2: Q2.B, R5.1
- new net Z: D1.P$2, D4.P$2, D5.P$2, R2.2
- net GND: now also D3.P$1, LED1.C, LED2.C, Q2.E, Q3.E; no longer D1.P$1, L1.C, L2.C, TR2.E
- net INPUT: now also D5.P$1, IC1.RA5; no longer D1.P$2, D2.P$1, D5.P$2, IC1.RA4, R2.2
- net N$10: now also LED1.A, R7.1; no longer L1.A, R6.1
- net N$11: now also R7.2; no longer R6.2
- net N$15: now also D2.A; no longer D3.A
- net N$16: now also R3.2; no longer R5.2
- net N$3: now also LED2.A; no longer L2.A
- net N$4: now also D2.C, R3.1, R4.2; no longer D3.C, R3.2, R5.1
- net N$6: now also Q3.B, R6.2; no longer R4.2, TR2.B
- net N$9: now also D3.P$2, Q3.C; no longer D4.P$2, TR2.C
- net OUTPUT: now also R6.1; no longer R4.1
- net POWER_CTRL: now also IC1.RA4, R5.2; no longer D5.P$1, IC1.RA5, Q1.G, R3.1
- net VCC: no longer D2.P$2
Other:
- note added: "CC-NC-BY-SA"
- note added: "June 2019 - Sixty four pixels ltd"
- note added: "LATCHBOX v1"
- moved on the sheet: BATT, C1, D1, D4, D5, ICSP, OUT, R1, R3, R4, R5, R6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

Commit message: sas
Parts:
- R1, R6, R7: value (none) -> 1k
- R2: value (none) -> 100r
- R4: value (none) -> 10k
Changed lines of the file:
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@@
 <part name="IC1" library="jasons_stuff" deviceset="PIC12F1822" device="SO08"/>
 <part name="D4" library="jasons_stuff" deviceset="0805DIODE" device=""/>
-<part name="R2" library="rcl" deviceset="R-EU_" device="R0805"/>
+<part name="R2" library="rcl" deviceset="R-EU_" device="R0805" value="100r"/>
 <part name="Q1" library="microbuilder" deviceset="MOSFET-P" device=""/>
 <part name="D1" library="jasons_stuff" deviceset="0805DIODE" device=""/>
@@
 <part name="P+2" library="supply1" deviceset="VCC" device=""/>
 <part name="P+3" library="supply1" deviceset="VCC" device=""/>
-<part name="R6" library="rcl" deviceset="R-EU_" device="R0805"/>
+<part name="R6" library="rcl" deviceset="R-EU_" device="R0805" value="1k"/>
 <part name="GND5" library="supply1" deviceset="GND" device=""/>
 <part name="D3" library="jasons_stuff" deviceset="0805DIODE" device=""/>
@@
 <part name="P+5" library="supply1" deviceset="VCC" device=""/>
 <part name="C3" library="rcl" deviceset="CPOL-EU" device="E2,5-6E"/>
-<part name="R4" library="rcl" deviceset="R-EU_" device="R0805"/>
+<part name="R4" library="rcl" deviceset="R-EU_" device="R0805" value="10k"/>
 <part name="GND6" library="supply1" deviceset="GND" device=""/>
 <part name="C2" library="rcl" deviceset="CPOL-EU" device="E2,5-6E"/>
@@
 <part name="LED2" library="led" deviceset="LED" device="3MM"/>
 <part name="LED1" library="led" deviceset="LED" device="3MM"/>
-<part name="R7" library="rcl" deviceset="R-EU_" device="R0805"/>
-<part name="R1" library="rcl" deviceset="R-EU_" device="R0805"/>
+<part name="R7" library="rcl" deviceset="R-EU_" device="R0805" value="1k"/>
+<part name="R1" library="rcl" deviceset="R-EU_" device="R0805" value="1k"/>
 <part name="GND8" library="supply1" deviceset="GND" device=""/>
 <part name="GND9" library="supply1" deviceset="GND" device=""/>
