File: latchbox-lite.sch (EAGLE design)
At the start: 28 parts, among them IC1 PIC12F1822SO08

Commit message: v2 possible
Parts:
- removed C3: (no value), rcl:CPOL-EUE2,5-6E
- removed Q3: (no value), transistor:MMBTA13LT1-NPN_DARL-SOT23-BEC
- removed R7: 1k, rcl:R-EU_R0805
- added D6, D7: 0805DIODE, jasons_stuff:0805DIODE
- added S1: (no value), switch-omron:31-XX
- C2: value (none) -> 4u7
- D1, D3: value 0805DIODE -> (none); device jasons_stuff:0805DIODE -> microbuilder:DIODESOD-123
- Q2: device transistor:MMBT3904LT1-NPN-SOT23-BEC -> transistor:MMBTA13LT1-NPN_DARL-SOT23-BEC
- R1: value 1k -> 100r
- R2: value 100r -> 1k
- R3: value (none) -> 10k
- R4: value 10k -> 4r7
- R5: value (none) -> 1k
Connections:
- removed net N: D1.P$1, Q1.G, Q2.C, R4.1
- removed net N$2: Q2.B, R5.1
- new net USB_POWER: D2.A, D3.A, R4.1
- net GND: now also D6.P$1, D7.P$1, S1.P; no longer C3.-, D3.P$1, D4.P$1, Q3.E
- net N$1: now also R1.1; no longer R2.1
- net N$10: now also R6.1; no longer R7.1
- net N$11: now also R6.2; no longer R7.2
- net N$12: now also D3.C, R2.2; no longer R1.2
- net N$14: now also D4.P$2, S1.S
- net N$15: now also D1.A; no longer D2.A
- net N$16: now also R4.2; no longer R3.2
- net N$3: now also R2.1; no longer R1.1
- net N$4: now also D1.C, R3.2; no longer C3.+, D2.C, R3.1, R4.2
- net N$6: now also Q2.B, R5.2; no longer Q3.B, R6.2
- net N$9: now also D7.P$2, Q2.C; no longer D3.P$2, Q3.C
- net OUTPUT: now also R5.1; no longer R6.1
- net POWER_CTRL: now also D4.P$1, Q1.G, R3.1; no longer R5.2
- net VCC: now also D2.C
- net Z: now also D6.P$2, R1.2; no longer D1.P$2, D4.P$2, R2.2
Other:
- note added: "August 2019 - Sixty four pixels ltd"
- note added: "LATCHBOX v2"
- note added: "RA1 periodically used as an input to detect USB power present"
- note added: "switch pulls gate of Q1 low when pressed, switching on power if running on battery"
- note added: "when MCU is running, POWER_CTRL is pulled low to keep power on RA3 is set to input with pull-up so further switch press can be detected without change to power status"
- note removed: "June 2019 - Sixty four pixels ltd"
- note removed: "LATCHBOX v1"
- moved on the sheet: C1, C2, D2, D4, D5, ICSP, IN, LED2, R1, R2, R3, R4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

Commit message: V3
Connections:
- net GND: now also IN.2; no longer IN.3
Other:
- note added: "LATCHBOX v3"
- note removed: "LATCHBOX v2"
Changed lines of the file:
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@@
 <sheet>
 <plain>
-<text x="10.16" y="71.12" size="5.08" layer="95">LATCHBOX v2</text>
+<text x="10.16" y="71.12" size="5.08" layer="95">LATCHBOX v3</text>
 <text x="10.16" y="63.5" size="5.08" layer="95">August 2019 - Sixty four pixels ltd</text>
 <text x="10.16" y="55.88" size="5.08" layer="95">CC-NC-BY-SA</text>
@@
 </segment>
 <segment>
-<pinref part="IN" gate="G$1" pin="3"/>
 <pinref part="GND3" gate="1" pin="GND"/>
-<wire x1="68.58" y1="226.06" x2="88.9" y2="226.06" width="0.1524" layer="91"/>
-<wire x1="88.9" y1="226.06" x2="88.9" y2="218.44" width="0.1524" layer="91"/>
+<wire x1="88.9" y1="231.14" x2="88.9" y2="218.44" width="0.1524" layer="91"/>
+<pinref part="IN" gate="G$1" pin="2"/>
+<wire x1="68.58" y1="231.14" x2="88.9" y2="231.14" width="0.1524" layer="91"/>
 </segment>
 <segment>

Commit message: V3 BOARD
Parts:
- removed D7: 0805DIODE, jasons_stuff:0805DIODE
- added Q3: (no value), transistor:MMBT3904LT1-NPN-SOT23-BEC
- added R7: 10k, rcl:R-EU_R0805
Connections:
- new net N$13: Q3.B, R7.2
- new net N$2: D3.A, Q1.G, Q3.C, R3.1
- net GND: now also D5.P$1, Q3.E; no longer D7.P$1
- net INPUT: now also D4.P$1; no longer D5.P$1
- net N$12: no longer D3.C
- net N$14: now also D3.C; no longer D4.P$2
- net N$9: now also D6.P$2; no longer D7.P$2
- net POWER_CTRL: now also R7.1; no longer D4.P$1, Q1.G, R3.1
- net USB_POWER: no longer D3.A
- net Z: now also D4.P$2; no longer D6.P$2
Other:
- note added: "October 2019 - Sixty four pixels ltd"
- note removed: "August 2019 - Sixty four pixels ltd"
- note removed: "RA1 periodically used as an input to detect USB power present"
- note removed: "switch pulls gate of Q1 low when pressed, switching on power if running on battery"
- note removed: "when MCU is running, POWER_CTRL is pulled low to keep power on RA3 is set to input with pull-up so further switch press can be detected without change to power status"
- moved on the sheet: D3, D4, D5, D6, S1

Commit message: V2 firmware
Parts:
- R7: value 10k -> 1k
Changed lines of the file:
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@@
 <part name="P+6" library="supply1" deviceset="VCC" device=""/>
 <part name="Q3" library="transistor" deviceset="*-NPN-" device="SOT23-BEC" technology="MMBT3904LT1"/>
-<part name="R7" library="rcl" deviceset="R-EU_" device="R0805" value="10k"/>
+<part name="R7" library="rcl" deviceset="R-EU_" device="R0805" value="1k"/>
 <part name="GND6" library="supply1" deviceset="GND" device=""/>
 <part name="GND10" library="supply1" deviceset="GND" device=""/>

Commit message: V4
Parts:
- D3: value (none) -> 0805DIODE; device microbuilder:DIODESOD-123 -> jasons_stuff:0805DIODE
Connections:
- net N$14: now also D3.P$2; no longer D3.C
- net N$2: now also D3.P$1; no longer D3.A
Other:
- note added: "LATCHBOX v4"
- note added: "November 2019 - Sixty four pixels ltd"
- note removed: "LATCHBOX v3"
- note removed: "October 2019 - Sixty four pixels ltd"
Changed lines of the file:
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@@
 <part name="GND6" library="supply1" deviceset="GND" device=""/>
 <part name="GND10" library="supply1" deviceset="GND" device=""/>
-<part name="D3" library="microbuilder" deviceset="DIODE" device="SOD-123"/>
+<part name="D3" library="jasons_stuff" deviceset="0805DIODE" device=""/>
 </parts>
 <sheets>
 <sheet>
 <plain>
-<text x="10.16" y="71.12" size="5.08" layer="95">LATCHBOX v3</text>
-<text x="10.16" y="63.5" size="5.08" layer="95">October 2019 - Sixty four pixels ltd</text>
+<text x="10.16" y="71.12" size="5.08" layer="95">LATCHBOX v4</text>
+<text x="10.16" y="63.5" size="5.08" layer="95">November 2019 - Sixty four pixels ltd</text>
 <text x="10.16" y="55.88" size="5.08" layer="95">CC-NC-BY-SA</text>
 </plain>
@@
 <instance part="GND6" gate="1" x="63.5" y="127"/>
 <instance part="GND10" gate="1" x="55.88" y="93.98"/>
-<instance part="D3" gate="G$1" x="55.88" y="129.54" rot="R270"/>
+<instance part="D3" gate="G$1" x="55.88" y="127" rot="R180"/>
 </instances>
 <busses>
@@
 <junction x="119.38" y="114.3"/>
 <pinref part="S1" gate="1" pin="S"/>
-<pinref part="D3" gate="G$1" pin="C"/>
-<wire x1="55.88" y1="127" x2="55.88" y2="114.3" width="0.1524" layer="91"/>
 <wire x1="55.88" y1="114.3" x2="55.88" y2="111.76" width="0.1524" layer="91"/>
 <wire x1="91.44" y1="114.3" x2="55.88" y2="114.3" width="0.1524" layer="91"/>
 <junction x="91.44" y="114.3"/>
 <junction x="55.88" y="114.3"/>
+<pinref part="D3" gate="G$1" pin="P$2"/>
+<wire x1="55.88" y1="114.3" x2="55.88" y2="126.492" width="0.1524" layer="91"/>
 </segment>
 </net>
@@
 <wire x1="63.5" y1="144.78" x2="63.5" y2="142.24" width="0.1524" layer="91"/>
 <junction x="63.5" y="144.78"/>
-<pinref part="D3" gate="G$1" pin="A"/>
-<wire x1="55.88" y1="144.78" x2="55.88" y2="132.08" width="0.1524" layer="91"/>
 <junction x="55.88" y="144.78"/>
-</segment>
-</net>
+<pinref part="D3" gate="G$1" pin="P$1"/>
+<wire x1="55.88" y1="144.78" x2="55.88" y2="131.572" width="0.1524" layer="91"/>
+</segment>
+</net>
