File: pcb-panel/latchbox-lite-stencil.brd (EAGLE design)
At the start: 137.4 x 87.9 mm, 235 parts, among them IC1 PIC12F1822SO08, IC2 PIC12F1822SO08, IC3 PIC12F1822SO08, IC4 PIC12F1822SO08, IC5 PIC12F1822SO08, IC6 PIC12F1822SO08, IC7 PIC12F1822SO08, IC8 PIC12F1822SO08

Commit message: stencil
Other:
- board size 137.4 x 87.9 mm -> 144 x 94 mm
